File: KiCad/led_clock.sch (KiCad schematic (older format))
At the start: 71 parts, among them P1 5V, SW1 SECONDS, SW2 MINUTES, SW3 HOURS, U1 74HCT4060, U10 74LS47, U11 74LS90, U12 74LS90, U13 74LS90, U14 74LS90, U15 74LS90, U16 74LS90, U2 74LS00, U3 74LS00, U4 74LS00, U5 74LS47, U6 74LS47, U7 74LS47, U8 74LS47, U9 74LS47, X1 32768Hz

Commit message: Add files for version 1.1
Signed-off-by: Sergey Kiselev <skiselev@gmail.com>
Parts:
- removed U1: 74HCT4060, symbol CD4060
- removed X1: 32768Hz, ~, symbol CRYSTAL
- added U1: 74HCT4060, My_Components:IC_DIP16_300, symbol 74HCT4060
- added Y1: 32768Hz, My_Components:Crystal_32K_Horiz, symbol Crystal
- C1, C10, C11, C12, C13, C14, C15, C16, C17, C2, C3, C4, C5, C6, C7, C8, C9: footprint ~ -> My_Components:Cap_Cer_762
- C18: footprint ~ -> My_Components:Cap_Cer_508
- C19: footprint ~ -> My_Components:C_Trim_Murata
- D1, D2, D3, D4: footprint ~ -> My_Components:LED_3mm
- DIS1, DIS2, DIS3, DIS4, DIS5, DIS6: footprint (none) -> My_Components:Display_LED7_DIP14_300
- HOLE1, HOLE2, HOLE3, HOLE4: footprint (none) -> My_Components:Hole_3mm
- P1: footprint (none) -> My_Components:Conn_Power_Jack_Circular_Pads
- R1, R10, R11, R2, R3, R4, R5, R6, R7, R8, R9: footprint ~ -> My_Components:Res_762
- RP1, RP2, RP3, RP4, RP5, RP6, U11, U12, U13, U14, U15, U16, U2, U3, U4: footprint ~ -> My_Components:IC_DIP14_300
- SW1, SW2, SW3: footprint ~ -> My_Components:Switch_SPDP_D2F
- U10, U5, U6, U7, U8, U9: footprint ~ -> My_Components:IC_DIP16_300
Other:
- moved on the sheet: C1, C10, C11, C12, C13, C14, C15, C16, C17, C18, C19, C2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

Commit message: Hide footprint fields in the schematic
Signed-off-by: Sergey Kiselev <skiselev@gmail.com>
Parts:
- C17: footprint My_Components:Cap_Cer_762 -> My_Components:Cap_Elec_Radial_6.3mm

Commit message: Use dual digit display
Signed-off-by: Sergey Kiselev <skiselev@gmail.com>
Parts:
- removed DIS1, DIS2, DIS3, DIS4, DIS5, DIS6: MAN1A, My_Components:Display_LED7_DIP14_300, symbol MAN1A
- added DIS1, DIS2, DIS3: HDSP-5521, symbol HDSP-5521
Connections:
- wire segments 485 -> 491
